Commit message: add first version of a pedestrian simulator

File: urdf/pedestrian.xacro (robot description, xacro)
@@ -8,5 +8,4 @@
   <xacro:property name="mass" value="1"/>
   <xacro:property name="PI" value="3.141592654"/>
-  <xacro:property name="test" value="$(arg t)"/>
   <link name="base_link">
     <collision>
